Commit message: updated repo with SLAM and world

File: urdf/amr.urdf (robot description, URDF)
Before this commit: robot amr, 6 links, 5 joints
Links:
- added link lidar_link, mass 0.2; collision cylinder length=0.04 radius=0.02; visual cylinder length=0.04 radius=0.02
Joints:
- added joint lidar_joint: type fixed, parent base_link, child lidar_link, origin xyz=0 0 0.0875 rpy=0 0 0
- joint left_wheel_joint: origin xyz=0 0.15 0 -> xyz=0 0.17 0
- joint right_wheel_joint: origin xyz=0 -0.15 0 -> xyz=0 -0.17 0
